File: PGA2040_Carrier.kicad_pcb (KiCad board)
At the start: 2 copper layers, 438.3 x 140.9 mm, 222 parts, among them J1 Conn_01x04_Pin, J2 Conn_01x04_Pin, U2 USBLC6-2SC6

Commit message: Add files via upload
Parts:
- J1, J2: value Conn_01x04_Pin -> Conn_01x05_Pin; footprint Connector_PinHeader_2.54mm:PinHeader_1x04_P2.54mm_Vertical -> Connector_PinHeader_2.54mm:PinHeader_1x05_P2.54mm_Vertical
- moved J1 427.3 mm to (465.6, 54.2), turned to -90 degrees
- moved J2 407.0 mm to (48.5, 54.0), turned to -90 degrees
Connections:
- J1 pad 1: VBUS_USB -> GND
- J1 pad 2: GND -> USB_DP
- J1 pad 4: USB_DP -> GND
- J2 pad 1: VBUS_USB -> GND
- J2 pad 2: GND -> USB_DP
- J2 pad 4: USB_DP -> GND
Routing:
- net USB_DP: track 471.3 -> 470.7 mm
